File: PCB+schematic/logan.kicad_pcb (KiCad board)
At the start: 2 copper layers, 91.5 x 54 mm, 11 parts, among them J1 Arduino DC Jack (6-12v), J2 SD Card, J3 BME280, J4 LoRa, J5 LoRa G pins

Commit message: update files
Parts:
- removed J3: BME280, Connector_PinHeader_2.54mm:PinHeader_1x04_P2.54mm_Vertical
- added A2: Arduino_Nano_v3.x, Module:Arduino_Nano, F.Cu at (192.8, 79.3)
Connections:
- A1 pad 1: /D1/TX -> /A0_TX
- A1 pad 23: /BME_SDA -> /A4
- A1 pad 24: /BME_SCL -> /A5
- A1 pad 8: /SD_CS -> /D5
- J2 pad 2: /MISO -> /SD_MISO
- J2 pad 3: /SCK -> /SD_SCK
- J2 pad 4: /MOSI -> /SD_MOSI
- J2 pad 6: +3.3V -> A1_3V3
Routing:
- net /NANO_VIN: track 42.0 -> 96.8 mm
- net /A0_TX: track 0.00 -> 54.0 mm
- net /SD_SCK: track 0.00 -> 42.3 mm
- net /MOSI: track 67.8 -> 29.6 mm
- net +3.3V: track 33.8 -> 0.00 mm
- net A1_3V3: track 0.00 -> 33.6 mm
- net /MISO: track 64.4 -> 31.2 mm
- net /SD_MISO: track 0.00 -> 29.6 mm
- net /SD_MOSI: track 0.00 -> 23.4 mm
- net /BME_SDA: track 21.2 -> 0.00 mm
- net /BME_SCL: track 21.0 -> 0.00 mm
- net /SCK: track 71.4 -> 50.9 mm
- net +5V: track 66.6 -> 49.9 mm
- net /~{A1_RESET}: track 0.00 -> 15.2 mm
- net /SD_CS: track 37.0 -> 21.8 mm
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Other:
- board size 91.5 x 54 mm -> 115.5 x 57.5 mm
