File: PCB+schematic/logan.kicad_pcb (KiCad board)
At the start: 2 copper layers, 115.5 x 57.5 mm, 11 parts, among them J1 Arduino DC Jack (6-12v), J2 SD Card, J4 LoRa, J5 LoRa G pins

Commit message: Long overdue folder structure update
Parts:
- added J6: Conn_01x08_Pin, Connector_PinSocket_2.54mm:PinSocket_1x08_P2.54mm_Vertical, F.Cu at (116.3, 104.8)
- moved H4 32.7 mm to (217.0, 124.5)
- moved H2 32.1 mm to (216.5, 73.0)
Routing:
- net /D6: track 0.00 -> 31.0 mm
- net /D7: track 0.00 -> 29.6 mm
- net /D9: track 0.00 -> 27.4 mm
- net /D8: track 0.00 -> 26.6 mm
Other:
- board size 115.5 x 57.5 mm -> 123 x 57.5 mm
