File: PCB+schematic/logan.kicad_sch (KiCad schematic)
At the start: 10 parts, among them J1 Arduino DC Jack (6-12v), J2 SD Card, J3 BME280, J4 LoRa, J5 LoRa G pins

Commit message: update files
Parts:
- removed J3: BME280, Connector_PinHeader_2.54mm:PinHeader_1x04_P2.54mm_Vertical, symbol Connector:Conn_01x04_Socket
- added A2: Arduino_Nano_v3.x, Module:Arduino_Nano, symbol MCU_Module:Arduino_Nano_v3.x
Connections:
- net +3.3V: no longer J2.6 (Pin_6)
- net Earth: now also A2.29 (GND), A2.4 (GND)
- net MISO: no longer J2.2 (Pin_2)
- net MOSI: no longer J2.4 (Pin_4)
- net NANO_VIN: now also A2.30 (VIN)
- net SCK: no longer J2.3 (Pin_3)
- net SD_CS: now also A2.7 (D4); no longer A1.8 (D5)
- net BME_SCL renamed A5
- net BME_SDA renamed A4
- net D1/TX renamed A0_TX
- net A0_TX: now also A2.2 (D0/RX)
- new net A1_+5V: A2.27 (+5V)
- new net A1_3V3: A2.17 (3V3), J2.6 (Pin_6)
- new net A1_A0: A2.19 (A0)
- new net A1_A1: A2.20 (A1)
- new net A1_A2: A2.21 (A2)
- new net A1_A3: A2.22 (A3)
- new net A1_A4: A2.23 (A4)
- new net A1_A5: A2.24 (A5)
- new net A1_A6: A2.25 (A6)
- new net A1_A7: A2.26 (A7)
- new net A1_AREF: A2.18 (AREF)
- new net A1_D10: A2.13 (D10)
- new net A1_D1/TX: A2.1 (D1/TX)
- new net A1_D2: A2.5 (D2)
- new net A1_D3: A2.6 (D3)
- new net A1_D5: A2.8 (D5)
- new net A1_D6: A2.9 (D6)
- new net A1_D7: A2.10 (D7)
- new net A1_D8: A2.11 (D8)
- new net A1_D9: A2.12 (D9)
- new net D5: A1.8 (D5)
- new net SD_MISO: A2.15 (D12), J2.2 (Pin_2)
- new net SD_MOSI: A2.14 (D11), J2.4 (Pin_4)
- new net SD_SCK: A2.16 (D13), J2.3 (Pin_3)
- new net ~{A1_RESET}: A2.28 (~{RESET}), A2.3 (~{RESET})
